Commit message: cameras added

File: src/robot_description/models/robot.urdf (robot description, URDF)
Before this commit: robot mobile_robot, 6 links, 5 joints
Links:
- added link camera_link; collision box size=0.0175 0.091 0.028; visual box size=0.0175 0.091 0.028
- added link camera_optical_link
Joints:
- added joint camera_joint: type fixed, parent base_link, child camera_link, origin xyz=${base_length/2} 0 0 rpy=0 0 0
- added joint camera_optical_joint: type fixed, parent camera_link, child camera_optical_link, origin xyz=0 0 0 rpy=${-pi/2} 0 ${-pi/2}

Commit message: camera tilted

File: src/robot_description/models/robot.urdf (robot description, URDF)
Before this commit: robot mobile_robot, 8 links, 7 joints
Joints:
- joint camera_joint: origin xyz=${base_length/2} 0 0 rpy=0 0 0 -> xyz=${base_length/2} 0 0 rpy=0 -0.37 0

Commit message: IMU and model state added

File: src/robot_description/models/robot.urdf (robot description, URDF)
Before this commit: robot mobile_robot, 8 links, 7 joints
Joints:
- joint imu_joint: origin xyz=-0.10 0 0.05 rpy=0 0 0 -> xyz=${base_length/2} 0 0 rpy=0 0 0
